Commit message: Update E190 bot URDF model

File: src/ros_robotics/urdf/e190_bot.urdf (robot description, URDF)
Before this commit: robot e190_bot, 3 links, 2 joints
Links:
- link base_link: mass @ -> 0.308; geometry collision cylinder length=0.03 radius=0.075; collision sphere radius=0.0125
- link left_wheel: mass @ -> 0.012; geometry collision cylinder length=0.008 radius=0.0335; visual cylinder length=0.008 radius=0.0335
- link right_wheel: mass @ -> 0.012; geometry collision cylinder length=0.008 radius=0.0335; visual cylinder length=0.008 radius=0.0335
Joints:
- joint joint_left_wheel: origin xyz=0 @ 0 rpy=0 0 0 -> xyz=0 0.07 0 rpy=0 0 0
- joint joint_right_wheel: origin xyz=0 -@ 0 rpy=0 0 0 -> xyz=0 -0.07 0 rpy=0 0 0
