Commit message: path planning done

File: src/e190_bot/urdf/pololu_romi.urdf (robot description, URDF)
Before this commit: robot pololu_romi, 2 links, 1 joints
Links:
- added link left_wheel, mass 0.5; collision cylinder length=0.008 radius=0.035; visual cylinder length=0.008 radius=0.035
- link base_link: geometry collision cylinder length=0.01 radius=0.0825; collision sphere radius=0.0127
Joints:
- added joint joint_left_wheel: type continuous, parent base_link, child left_wheel, origin xyz=0 0.0825 0.0127 rpy=0 0 0, axis 0 1 0
- joint joint_right_wheel: origin xyz=0 -0.0825 0 rpy=0 0 0 -> xyz=0 -0.0825 0.0127 rpy=0 0 0
